File: pcb_base.sch (KiCad schematic (older format))
At the start: 4 parts, among them U1 ATMEGA32U4, X1 XTAL_GND

Commit message: add vcc decoupling capacitors
Parts:
- added C3, C4, C5, C6: 0.1u, symbol Device:C_Small
- added C7: 4.7u, symbol Device:C_Small
Connections:
- net labels added: VCC
- wire segments 14 -> 34
Changed lines of the file:
@@
 EESchema Schematic File Version 4
+LIBS:pcb_base-cache
 EELAYER 26 0
 EELAYER END
@@
 	2500 3950 2500 4150
 Connection ~ 2500 4150
+$Comp
+L Device:C_Small C3
+U 1 1 5BAEBF1A
+P 1650 1650
+F 0 "C3" H 1742 1696 50  0000 L CNN
+F 1 "0.1u" H 1742 1605 50  0000 L CNN
+F 2 "" H 1650 1650 50  0001 C CNN
+F 3 "~" H 1650 1650 50  0001 C CNN
+	1    1650 1650
+	1    0    0    -1
+$EndComp
+$Comp
+L Device:C_Small C4
+U 1 1 5BAEBF7F
+P 2000 1650
+F 0 "C4" H 2092 1696 50  0000 L CNN
+F 1 "0.1u" H 2092 1605 50  0000 L CNN
+F 2 "" H 2000 1650 50  0001 C CNN
+F 3 "~" H 2000 1650 50  0001 C CNN
+	1    2000 1650
+	1    0    0    -1
+$EndComp
+$Comp
+L Device:C_Small C5
+U 1 1 5BAEBFA3
+P 2350 1650
+F 0 "C5" H 2442 1696 50  0000 L CNN
+F 1 "0.1u" H 2442 1605 50  0000 L CNN
+F 2 "" H 2350 1650 50  0001 C CNN
+F 3 "~" H 2350 1650 50  0001 C CNN
+	1    2350 1650
+	1    0    0    -1
+$EndComp
+$Comp
+L Device:C_Small C6
+U 1 1 5BAEBFC6
+P 2700 1650
+F 0 "C6" H 2792 1696 50  0000 L CNN
+F 1 "0.1u" H 2792 1605 50  0000 L CNN
+F 2 "" H 2700 1650 50  0001 C CNN
+F 3 "~" H 2700 1650 50  0001 C CNN
+	1    2700 1650
+	1    0    0    -1
+$EndComp
+$Comp
+L Device:C_Small C7
+U 1 1 5BAEBFED
+P 3050 1650
+F 0 "C7" H 3142 1696 50  0000 L CNN
+F 1 "4.7u" H 3142 1605 50  0000 L CNN
+F 2 "" H 3050 1650 50  0001 C CNN
+F 3 "~" H 3050 1650 50  0001 C CNN
+	1    3050 1650
+	1    0    0    -1
+$EndComp
+Wire Wire Line
+	1650 1550 1650 1450
+Wire Wire Line
+	1650 1450 2000 1450
+Wire Wire Line
+	2000 1450 2000 1550
+Wire Wire Line
+	2000 1450 2350 1450
+Wire Wire Line
+	2350 1450 2350 1550
+Connection ~ 2000 1450
+Wire Wire Line
+	2350 1450 2700 1450
+Wire Wire Line
+	2700 1450 2700 1550
+Connection ~ 2350 1450
+Wire Wire Line
+	2700 1450 3050 1450
+Wire Wire Line
+	3050 1450 3050 1550
+Connection ~ 2700 1450
+Wire Wire Line
+	1650 1750 1650 1850
+Wire Wire Line
+	1650 1850 2000 1850
+Wire Wire Line
+	2000 1850 2000 1750
+Wire Wire Line
+	2000 1850 2350 1850
+Wire Wire Line
+	2350 1850 2350 1750
+Connection ~ 2000 1850
+Wire Wire Line
+	2350 1850 2700 1850
+Wire Wire Line
+	2700 1850 2700 1750
+Connection ~ 2350 1850
+Wire Wire Line
+	2700 1850 3050 1850
+Wire Wire Line
+	3050 1850 3050 1750
+Connection ~ 2700 1850
+$Comp
+L power:VCC #PWR?
+U 1 1 5BAEDB30
+P 1650 1300
+F 0 "#PWR?" H 1650 1150 50  0001 C CNN
+F 1 "VCC" H 1667 1473 50  0000 C CNN
+F 2 "" H 1650 1300 50  0001 C CNN
+F 3 "" H 1650 1300 50  0001 C CNN
+	1    1650 1300
+	1    0    0    -1
+$EndComp
+$Comp
+L power:GND #PWR?
+U 1 1 5BAEDBB3
+P 1650 2000
+F 0 "#PWR?" H 1650 1750 50  0001 C CNN
+F 1 "GND" H 1655 1827 50  0000 C CNN
+F 2 "" H 1650 2000 50  0001 C CNN
+F 3 "" H 1650 2000 50  0001 C CNN
+	1    1650 2000
+	1    0    0    -1
+$EndComp
+Wire Wire Line
+	1650 1450 1650 1300
+Connection ~ 1650 1450
+Wire Wire Line
+	1650 1850 1650 2000
+Connection ~ 1650 1850
 $EndSCHEMATC

Commit message: add a reset switch
Parts:
- added R1: 10k, symbol Device:R
- added SW1: SW_PUSH, symbol keyboard_parts:SW_PUSH
Connections:
- wire segments 34 -> 39
Changed lines of the file:
@@
 	1650 1450 1650 1300
 Connection ~ 1650 1450
+$Comp
+L keyboard_parts:SW_PUSH SW1
+U 1 1 5BAEE77B
+P 2900 3650
+F 0 "SW1" H 2900 3800 50  0000 C CNN
+F 1 "SW_PUSH" H 2900 3550 50  0000 C CNN
+F 2 "" H 2900 3650 60  0000 C CNN
+F 3 "" H 2900 3650 60  0000 C CNN
+	1    2900 3650
+	1    0    0    -1
+$EndComp
+$Comp
+L Device:R R1
+U 1 1 5BAEE9B2
+P 2850 3400
+F 0 "R1" V 2750 3400 50  0000 C CNN
+F 1 "10k" V 2850 3400 50  0000 C CNN
+F 2 "" V 2780 3400 50  0001 C CNN
+F 3 "~" H 2850 3400 50  0001 C CNN
+	1    2850 3400
+	0    1    1    0
+$EndComp
 Wire Wire Line
-	1650 1850 1650 2000
-Connection ~ 1650 1850
+	4000 3650 3350 3650
+Wire Wire Line
+	3000 3400 3350 3400
+Wire Wire Line
+	3350 3400 3350 3650
+Connection ~ 3350 3650
+Wire Wire Line
+	3350 3650 3200 3650
+$Comp
+L power:VCC #PWR?
+U 1 1 5BAEF6A8
+P 2300 3400
+F 0 "#PWR?" H 2300 3250 50  0001 C CNN
+F 1 "VCC" V 2318 3527 50  0000 L CNN
+F 2 "" H 2300 3400 50  0001 C CNN
+F 3 "" H 2300 3400 50  0001 C CNN
+	1    2300 3400
+	0    -1   -1   0
+$EndComp
+$Comp
+L power:GND #PWR?
+U 1 1 5BAEF752
+P 2300 3650
+F 0 "#PWR?" H 2300 3400 50  0001 C CNN
+F 1 "GND" V 2305 3522 50  0000 R CNN
+F 2 "" H 2300 3650 50  0001 C CNN
+F 3 "" H 2300 3650 50  0001 C CNN
+	1    2300 3650
+	0    1    1    0
+$EndComp
+Wire Wire Line
+	2700 3400 2300 3400
+Wire Wire Line
+	2600 3650 2300 3650
 $EndSCHEMATC

Commit message: add reset resistor
Parts:
- added R?: 10k, symbol Device:R
Connections:
- wire segments 39 -> 41
Changed lines of the file:
@@
 Wire Wire Line
 	2600 3650 2300 3650
+$Comp
+L Device:R R?
+U 1 1 5BAF06AC
+P 6500 3550
+F 0 "R?" V 6400 3550 50  0000 C CNN
+F 1 "10k" V 6500 3550 50  0000 C CNN
+F 2 "" V 6430 3550 50  0001 C CNN
+F 3 "~" H 6500 3550 50  0001 C CNN
+	1    6500 3550
+	0    1    1    0
+$EndComp
+$Comp
+L power:GND #PWR?
+U 1 1 5BAF06E3
+P 6800 3550
+F 0 "#PWR?" H 6800 3300 50  0001 C CNN
+F 1 "GND" V 6805 3422 50  0000 R CNN
+F 2 "" H 6800 3550 50  0001 C CNN
+F 3 "" H 6800 3550 50  0001 C CNN
+	1    6800 3550
+	0    -1   -1   0
+$EndComp
+Wire Wire Line
+	6150 3550 6350 3550
+Wire Wire Line
+	6650 3550 6800 3550
 $EndSCHEMATC

Commit message: ground the ground and use vcc for the vccs
Parts:
- gave numbers to parts that had none: 1
Connections:
- wire segments 41 -> 47
Changed lines of the file:
@@
 	2600 3650 2300 3650
 $Comp
-L Device:R R?
+L Device:R R2
 U 1 1 5BAF06AC
 P 6500 3550
-F 0 "R?" V 6400 3550 50  0000 C CNN
+F 0 "R2" V 6600 3550 50  0000 C CNN
 F 1 "10k" V 6500 3550 50  0000 C CNN
 F 2 "" V 6430 3550 50  0001 C CNN
@@
 Wire Wire Line
 	6650 3550 6800 3550
+$Comp
+L power:GND #PWR?
+U 1 1 5BAF16C8
+P 6350 4550
+F 0 "#PWR?" H 6350 4300 50  0001 C CNN
+F 1 "GND" V 6355 4422 50  0000 R CNN
+F 2 "" H 6350 4550 50  0001 C CNN
+F 3 "" H 6350 4550 50  0001 C CNN
+	1    6350 4550
+	0    -1   -1   0
+$EndComp
+$Comp
+L power:GND #PWR?
+U 1 1 5BAF16EB
+P 6350 2550
+F 0 "#PWR?" H 6350 2300 50  0001 C CNN
+F 1 "GND" V 6355 2422 50  0000 R CNN
+F 2 "" H 6350 2550 50  0001 C CNN
+F 3 "" H 6350 2550 50  0001 C CNN
+	1    6350 2550
+	0    -1   -1   0
+$EndComp
+$Comp
+L power:GND #PWR?
+U 1 1 5BAF170E
+P 6300 3350
+F 0 "#PWR?" H 6300 3100 50  0001 C CNN
+F 1 "GND" V 6305 3222 50  0000 R CNN
+F 2 "" H 6300 3350 50  0001 C CNN
+F 3 "" H 6300 3350 50  0001 C CNN
+	1    6300 3350
+	0    -1   -1   0
+$EndComp
+$Comp
+L power:VCC #PWR?
+U 1 1 5BAF1826
+P 6650 2450
+F 0 "#PWR?" H 6650 2300 50  0001 C CNN
+F 1 "VCC" V 6667 2578 50  0000 L CNN
+F 2 "" H 6650 2450 50  0001 C CNN
+F 3 "" H 6650 2450 50  0001 C CNN
+	1    6650 2450
+	0    1    1    0
+$EndComp
+$Comp
+L power:VCC #PWR?
+U 1 1 5BAF1861
+P 7050 3450
+F 0 "#PWR?" H 7050 3300 50  0001 C CNN
+F 1 "VCC" V 7067 3578 50  0000 L CNN
+F 2 "" H 7050 3450 50  0001 C CNN
+F 3 "" H 7050 3450 50  0001 C CNN
+	1    7050 3450
+	0    1    1    0
+$EndComp
+$Comp
+L power:VCC #PWR?
+U 1 1 5BAF1884
+P 6600 4450
+F 0 "#PWR?" H 6600 4300 50  0001 C CNN
+F 1 "VCC" V 6617 4578 50  0000 L CNN
+F 2 "" H 6600 4450 50  0001 C CNN
+F 3 "" H 6600 4450 50  0001 C CNN
+	1    6600 4450
+	0    1    1    0
+$EndComp
+Wire Wire Line
+	6150 2550 6350 2550
+Wire Wire Line
+	6150 2450 6650 2450
+Wire Wire Line
+	6150 3350 6300 3350
+Wire Wire Line
+	6150 3450 7050 3450
+Wire Wire Line
+	6150 4450 6600 4450
+Wire Wire Line
+	6150 4550 6350 4550
 $EndSCHEMATC

Commit message: add usb c support for hro connector
Parts:
- added R3, R4: 5.1k, symbol Device:R
- added R6, R7: 22, symbol Device:R
- added USB1: HRO-TYPE-C-31-M-12, symbol Type-C:HRO-TYPE-C-31-M-12
Connections:
- wire segments 47 -> 75
Changed lines of the file:
@@
 Wire Wire Line
 	6150 4550 6350 4550
+$Comp
+L Type-C:HRO-TYPE-C-31-M-12 USB1
+U 1 1 5BB2C3EA
+P 1600 6250
+F 0 "USB1" H 1431 7047 60  0000 C CNN
+F 1 "HRO-TYPE-C-31-M-12" H 1431 6941 60  0000 C CNN
+F 2 "" H 1600 6250 60  0001 C CNN
+F 3 "" H 1600 6250 60  0001 C CNN
+	1    1600 6250
+	1    0    0    -1
+$EndComp
+$Comp
+L power:VCC #PWR?
+U 1 1 5BB2BAAD
+P 2850 5800
+F 0 "#PWR?" H 2850 5650 50  0001 C CNN
+F 1 "VCC" V 2867 5928 50  0000 L CNN
+F 2 "" H 2850 5800 50  0001 C CNN
+F 3 "" H 2850 5800 50  0001 C CNN
+	1    2850 5800
+	0    1    1    0
+$EndComp
+Wire Wire Line
+	1700 5800 2050 5800
+$Comp
+L power:GND #PWR?
+U 1 1 5BB2C548
+P 2100 5700
+F 0 "#PWR?" H 2100 5450 50  0001 C CNN
+F 1 "GND" V 2105 5572 50  0000 R CNN
+F 2 "" H 2100 5700 50  0001 C CNN
+F 3 "" H 2100 5700 50  0001 C CNN
+	1    2100 5700
+	0    -1   -1   0
+$EndComp
+Wire Wire Line
+	1700 5700 1850 5700
+$Comp
+L Device:R R3
+U 1 1 5BB2D3AA
+P 2300 6750
+F 0 "R3" H 2230 6704 50  0000 R CNN
+F 1 "5.1k" V 2300 6850 50  0000 R CNN
+F 2 "" V 2230 6750 50  0001 C CNN
+F 3 "~" H 2300 6750 50  0001 C CNN
+	1    2300 6750
+	-1   0    0    1
+$EndComp
+$Comp
+L Device:R R4
+U 1 1 5BB2D42C
+P 2600 6750
+F 0 "R4" H 2750 6700 50  0000 R CNN
+F 1 "5.1k" V 2600 6850 50  0000 R CNN
+F 2 "" V 2530 6750 50  0001 C CNN
+F 3 "~" H 2600 6750 50  0001 C CNN
+	1    2600 6750
+	1    0    0    1
+$EndComp
+Wire Wire Line
+	1700 6700 2050 6700
+Wire Wire Line
+	2050 6700 2050 5800
+Connection ~ 2050 5800
+Wire Wire Line
+	2050 5800 2850 5800
+Wire Wire Line
+	1700 6800 1850 6800
+Wire Wire Line
+	1850 6800 1850 5700
+Connection ~ 1850 5700
+Wire Wire Line
+	1850 5700 2100 5700
+Wire Wire Line
+	1700 6900 1850 6900
+Wire Wire Line
+	1850 6900 1850 6800
+Connection ~ 1850 6800
+$Comp
+L power:GND #PWR?
+U 1 1 5BB32527
+P 1850 7100
+F 0 "#PWR?" H 1850 6850 50  0001 C CNN
+F 1 "GND" H 1855 6927 50  0000 C CNN
+F 2 "" H 1850 7100 50  0001 C CNN
+F 3 "" H 1850 7100 50  0001 C CNN
+	1    1850 7100
+	1    0    0    -1
+$EndComp
+Wire Wire Line
+	1850 6900 1850 7100
+Connection ~ 1850 6900
+Wire Wire Line
+	1700 6600 2300 6600
+Wire Wire Line
+	1850 6900 2300 6900
+Wire Wire Line
+	1700 6000 2600 6000
+Wire Wire Line
+	2600 6000 2600 6600
+Wire Wire Line
+	2300 6900 2600 6900
+Connection ~ 2300 6900
+$Comp
+L Device:R R6
+U 1 1 5BB39165
+P 3350 6400
+F 0 "R6" V 3250 6400 50  0000 R CNN
+F 1 "22" V 3350 6500 50  0000 R CNN
+F 2 "" V 3280 6400 50  0001 C CNN
+F 3 "~" H 3350 6400 50  0001 C CNN
+	1    3350 6400
+	0    -1   -1   0
+$EndComp
+$Comp
+L Device:R R7
+U 1 1 5BB391C5
+P 3350 6100
+F 0 "R7" V 3250 6100 50  0000 R CNN
+F 1 "22" V 3350 6200 50  0000 R CNN
+F 2 "" V 3280 6100 50  0001 C CNN
+F 3 "~" H 3350 6100 50  0001 C CNN
+	1    3350 6100
+	0    -1   -1   0
+$EndComp
+Wire Wire Line
+	1700 6200 2150 6200
+Wire Wire Line
+	3100 6200 3100 6100
+Wire Wire Line
+	3100 6100 3200 6100
+Wire Wire Line
+	1700 6300 2200 6300
+Wire Wire Line
+	3100 6300 3100 6400
+Wire Wire Line
+	3100 6400 3200 6400
+Wire Wire Line
+	1700 6100 2200 6100
+Wire Wire Line
+	2200 6100 2200 6300
+Connection ~ 2200 6300
+Wire Wire Line
+	2200 6300 3100 6300
+Wire Wire Line
+	1700 6400 2150 6400
+Wire Wire Line
+	2150 6400 2150 6200
+Connection ~ 2150 6200
+Wire Wire Line
+	2150 6200 3100 6200
 $EndSCHEMATC

Commit message: add missing vcc and grnd connections
Parts:
- added C8: 1uF, symbol Device:C_Small
Connections:
- net labels added: D+, D-
- wire segments 75 -> 87
Changed lines of the file:
@@
 Wire Wire Line
 	2150 6200 3100 6200
+$Comp
+L Device:C_Small C8
+U 1 1 5BB2D59B
+P 3600 2950
+F 0 "C8" V 3450 2950 50  0000 C CNN
+F 1 "1uF" V 3750 2950 50  0000 C CNN
+F 2 "" H 3600 2950 50  0001 C CNN
+F 3 "~" H 3600 2950 50  0001 C CNN
+	1    3600 2950
+	0    1    1    0
+$EndComp
+$Comp
+L power:GND #PWR?
+U 1 1 5BB2D709
+P 3200 2950
+F 0 "#PWR?" H 3200 2700 50  0001 C CNN
+F 1 "GND" V 3205 2822 50  0000 R CNN
+F 2 "" H 3200 2950 50  0001 C CNN
+F 3 "" H 3200 2950 50  0001 C CNN
+	1    3200 2950
+	0    1    1    0
+$EndComp
+Wire Wire Line
+	4000 2950 3700 2950
+Wire Wire Line
+	3500 2950 3350 2950
+Wire Wire Line
+	4000 2850 3350 2850
+Wire Wire Line
+	3350 2850 3350 2950
+Connection ~ 3350 2950
+Wire Wire Line
+	3350 2950 3200 2950
+Wire Wire Line
+	1650 2000 1650 1850
+Connection ~ 1650 1850
+Text Label 3500 6100 0    50   ~ 0
+D+
+Text Label 3500 6400 0    50   ~ 0
+D-
+Text Label 4000 2750 2    50   ~ 0
+D+
+Text Label 4000 2650 2    50   ~ 0
+D-
+$Comp
+L power:VCC #PWR?
+U 1 1 5BB35CA1
+P 3250 2550
+F 0 "#PWR?" H 3250 2400 50  0001 C CNN
+F 1 "VCC" V 3268 2677 50  0000 L CNN
+F 2 "" H 3250 2550 50  0001 C CNN
+F 3 "" H 3250 2550 50  0001 C CNN
+	1    3250 2550
+	0    -1   -1   0
+$EndComp
+$Comp
+L power:GND #PWR?
+U 1 1 5BB39D94
+P 3750 3850
+F 0 "#PWR?" H 3750 3600 50  0001 C CNN
+F 1 "GND" V 3755 3722 50  0000 R CNN
+F 2 "" H 3750 3850 50  0001 C CNN
+F 3 "" H 3750 3850 50  0001 C CNN
+	1    3750 3850
+	0    1    1    0
+$EndComp
+$Comp
+L power:VCC #PWR?
+U 1 1 5BB39DC3
+P 3900 3750
+F 0 "#PWR?" H 3900 3600 50  0001 C CNN
+F 1 "VCC" V 3918 3877 50  0000 L CNN
+F 2 "" H 3900 3750 50  0001 C CNN
+F 3 "" H 3900 3750 50  0001 C CNN
+	1    3900 3750
+	0    -1   -1   0
+$EndComp
+Wire Wire Line
+	4000 3850 3750 3850
+Wire Wire Line
+	4000 3750 3900 3750
+Wire Wire Line
+	4000 3050 3750 3050
+Wire Wire Line
+	3750 2550 3250 2550
+Wire Wire Line
+	4000 2550 3750 2550
+Connection ~ 3750 2550
+Wire Wire Line
+	3750 3050 3750 2550
 $EndSCHEMATC
